Commit message: Xacro implementasjon i urdf-filen

File: src/joint_description/urdf/joint_model.urdf (robot description, URDF)
Before this commit: robot joint_model, 5 links, 4 joints
Links:
- link angle_link: geometry visual box size=${indicator_length} ${indicator_width} ${indicator_width}
- link rotor_link: geometry visual cylinder length=${rotor_length} radius=${rotor_radius}
- link stator_link: geometry visual box size=${stator_size} ${stator_size} ${stator_size}
Joints:
- removed joint indicator
- added joint indicator_joint: type fixed, parent rotor_link, child angle_link, origin xyz=${indicator_length/2} 0 ${rotor_length/2 + indicator_width/2} rpy=0 0 0
- joint angle_joint: origin xyz=0 0 0.056 rpy=0 0 0 -> xyz=0 0 ${stator_size/2 + rotor_length/2} rpy=0 0 0
- joint stator_joint: origin xyz=0 0 0.051 rpy=0 0 0 -> xyz=0 0 ${stator_size/2} rpy=0 0 0

Commit message: Lagde en makro-fil men generalisert kode

File: src/joint_description/urdf/joint_model.urdf (robot description, URDF)
Before this commit: robot joint_model, 5 links, 4 joints
Links:
- removed link angle_link
- removed link base_link
- removed link rotor_link
- removed link stator_link
Joints:
- removed joint angle_joint
- removed joint base_joint
- removed joint indicator_joint
- removed joint stator_joint
